Commit message: change inertia

File: uuv_descriptions/urdf/rexrov_base.xacro (robot description, xacro)
@@ -37,5 +37,5 @@
         <mass value="${mass}"/>
         <origin xyz="0 0 0"/>
-        <inertia ixx="525.39" ixy="1.44" ixz="33.41" iyy="794.20" iyz="2.6" izz="691.23"/>
+        <inertia ixx="2760.99" ixy="29.02" ixz="20.94" iyy="5161.46" iyz="29.39" izz="4332.90"/>
       </inertial>
       <visual>
