Commit message: change thrusters positions

File: uuv_descriptions/urdf/rexrov_actuators.xacro (robot description, xacro)
@@ -27,26 +27,26 @@
   </xacro:macro>
   <xacro:thruster_macro namespace="${namespace}" thruster_id="0">
-    <origin xyz="-0.890895 0.334385 0.528822" rpy="${0*d2r} ${-74.53*d2r} ${-53.21*d2r}"/>
+    <origin xyz="-0.76574 0.570 0.1577" rpy="${0*d2r} ${70*d2r} ${0*d2r}"/>
   </xacro:thruster_macro>
   <xacro:thruster_macro namespace="${namespace}" thruster_id="1">
-    <origin xyz="-0.890895 -0.334385 0.528822" rpy="${0*d2r} ${-74.53*d2r} ${53.21*d2r}"/>
+    <origin xyz="-0.76574 -0.570 0.1577" rpy="${0*d2r} ${-70*d2r} ${0*d2r}"/>
   </xacro:thruster_macro>
   <xacro:thruster_macro namespace="${namespace}" thruster_id="2">
-    <origin xyz="0.890895 0.334385 0.528822" rpy="${0*d2r} ${-105.47*d2r} ${53.21*d2r}"/>
+    <origin xyz="0.76574 0.570 0.1577" rpy="${0*d2r} ${110*d2r} ${0*d2r}"/>
   </xacro:thruster_macro>
   <xacro:thruster_macro namespace="${namespace}" thruster_id="3">
-    <origin xyz="0.890895 -0.334385 0.528822" rpy="${0*d2r} ${-105.47*d2r} ${-53.21*d2r}"/>
+    <origin xyz="0.76574 -0.570 0.1577" rpy="${0*d2r} ${-110*d2r} ${0*d2r}"/>
   </xacro:thruster_macro>
   <xacro:thruster_macro namespace="${namespace}" thruster_id="4">
-    <origin xyz="-0.412125 0.505415 0.129" rpy="${0*d2r} ${0*d2r} ${45*d2r}"/>
+    <origin xyz="-1.19239 0.56425 0.94606" rpy="${0*d2r} ${0*d2r} ${45*d2r}"/>
   </xacro:thruster_macro>
   <xacro:thruster_macro namespace="${namespace}" thruster_id="5">
-    <origin xyz="-0.412125 -0.505415 0.129" rpy="${0*d2r} ${0*d2r} ${-45*d2r}"/>
+    <origin xyz="-1.19239 -0.56425 0.94606" rpy="${0*d2r} ${0*d2r} ${-45*d2r}"/>
   </xacro:thruster_macro>
   <xacro:thruster_macro namespace="${namespace}" thruster_id="6">
-    <origin xyz="0.412125 0.505415 0.129" rpy="${0*d2r} ${0*d2r} ${135*d2r}"/>
+    <origin xyz="1.22921 0.56425 0.94606" rpy="${0*d2r} ${0*d2r} ${135*d2r}"/>
   </xacro:thruster_macro>
   <xacro:thruster_macro namespace="${namespace}" thruster_id="7">
-    <origin xyz="0.412125 -0.505415 0.129" rpy="${0*d2r} ${0*d2r} ${-135*d2r}"/>
+    <origin xyz="1.229215 -0.56425 0.94606" rpy="${0*d2r} ${0*d2r} ${-135*d2r}"/>
   </xacro:thruster_macro>
 </robot>

File: uuv_descriptions/urdf/rexrov_base.xacro (robot description, xacro)
@@ -42,27 +42,27 @@
         <origin xyz="0 0 0" rpy="0 0 0"/>
         <geometry>
-          <mesh filename="${visual_mesh_file}" scale="1 1 1"/>
+          <mesh filename="${visual_mesh_file}" scale="1.4 1.27 1.67"/>
         </geometry>
       </visual>
       <!-- bottom plate -->
       <collision>
-        <origin xyz="0 0 -0.75" rpy="0 0 0"/>
+        <origin xyz="0 0 -0.85" rpy="0 0 0"/>
         <geometry>
-          <box size="2.56 1.50 0.10"/>
+          <box size="3.598 1.905 0.10"/>
         </geometry>
       </collision>
       <!-- top plate -->
       <collision>
-        <origin xyz="0 0 0.60" rpy="0 0 0"/>
-        <geometry><box size="2.56 1.50 0.40"/></geometry>
+        <origin xyz="0 0 0.70" rpy="0 0 0"/>
+        <geometry><box size="3.598 1.905 0.40"/></geometry>
       </collision>
       <!-- left / right sides -->
       <collision>
-        <origin xyz="-0.20 0.70 -0.15" rpy="0 0 0"/>
-        <geometry><box size="2.20 0.10 1.10"/></geometry>
+        <origin xyz="-0.20 0.90 -0.15" rpy="0 0 0"/>
+        <geometry><box size="3.40 0.10 1.50"/></geometry>
       </collision>
       <collision>
-        <origin xyz="-0.20 -0.70 -0.15" rpy="0 0 0"/>
-        <geometry><box size="2.20 0.10 1.10"/></geometry>
+        <origin xyz="-0.20 -0.90 -0.15" rpy="0 0 0"/>
+        <geometry><box size="3.40 0.10 1.50"/></geometry>
       </collision>
     </link>

Commit message: change proportions

File: uuv_descriptions/urdf/rexrov_actuators.xacro (robot description, xacro)
@@ -27,14 +27,14 @@
   </xacro:macro>
   <xacro:thruster_macro namespace="${namespace}" thruster_id="0">
-    <origin xyz="-0.76574 0.570 0.577" rpy="${0*d2r} ${70*d2r} ${0*d2r}"/>
+    <origin xyz="-0.76574 0.570 0.577" rpy="${-70*d2r} ${0*d2r} ${0*d2r}"/>
   </xacro:thruster_macro>
   <xacro:thruster_macro namespace="${namespace}" thruster_id="1">
-    <origin xyz="-0.76574 -0.570 0.577" rpy="${0*d2r} ${-70*d2r} ${0*d2r}"/>
+    <origin xyz="-0.76574 -0.570 0.577" rpy="${-70*d2r} ${0*d2r} ${0*d2r}"/>
   </xacro:thruster_macro>
   <xacro:thruster_macro namespace="${namespace}" thruster_id="2">
-    <origin xyz="0.76574 0.570 0.577" rpy="${0*d2r} ${110*d2r} ${0*d2r}"/>
+    <origin xyz="0.76574 0.570 0.577" rpy="${-110*d2r} ${0*d2r} ${0*d2r}"/>
   </xacro:thruster_macro>
   <xacro:thruster_macro namespace="${namespace}" thruster_id="3">
-    <origin xyz="0.76574 -0.570 0.577" rpy="${0*d2r} ${-110*d2r} ${0*d2r}"/>
+    <origin xyz="0.76574 -0.570 0.577" rpy="${-110*d2r} ${0*d2r} ${0*d2r}"/>
   </xacro:thruster_macro>
   <xacro:thruster_macro namespace="${namespace}" thruster_id="4">

File: uuv_descriptions/urdf/rexrov_base.xacro (robot description, xacro)
@@ -39,4 +39,10 @@
         <inertia ixx="2760.99" ixy="29.02" ixz="20.94" iyy="5161.46" iyz="29.39" izz="4332.90"/>
       </inertial>
+      <visual>
+        <origin xyz="0 0 0" rpy="0 0 0"/>
+        <geometry>
+          <mesh filename="${visual_mesh_file}" scale="1.4 1.27 1.25"/>
+        </geometry>
+      </visual>
       <!-- bottom plate -->
       <collision>

Commit message: fix thruster angles

File: uuv_descriptions/urdf/rexrov_actuators.xacro (robot description, xacro)
@@ -26,15 +26,15 @@
     </xacro:thruster_module_first_order_basic_fcn_macro>
   </xacro:macro>
-  <xacro:thruster_macro namespace="${namespace}" thruster_id="0">
-    <origin xyz="-0.76574 0.570 0.577" rpy="${-70*d2r} ${0*d2r} ${0*d2r}"/>
+ <xacro:thruster_macro namespace="${namespace}" thruster_id="0">
+    <origin xyz="-0.76574 0.570 0.577" rpy="${0*d2r} ${-70*d2r} ${-90*d2r}"/>
   </xacro:thruster_macro>
   <xacro:thruster_macro namespace="${namespace}" thruster_id="1">
-    <origin xyz="-0.76574 -0.570 0.577" rpy="${-70*d2r} ${0*d2r} ${0*d2r}"/>
+    <origin xyz="-0.76574 -0.570 0.577" rpy="${0*d2r} ${-70*d2r} ${90*d2r}"/>
   </xacro:thruster_macro>
   <xacro:thruster_macro namespace="${namespace}" thruster_id="2">
-    <origin xyz="0.76574 0.570 0.577" rpy="${-110*d2r} ${0*d2r} ${0*d2r}"/>
+    <origin xyz="0.76574 0.570 0.577" rpy="${0*d2r} ${-110*d2r} ${90*d2r}"/>
   </xacro:thruster_macro>
   <xacro:thruster_macro namespace="${namespace}" thruster_id="3">
-    <origin xyz="0.76574 -0.570 0.577" rpy="${-110*d2r} ${0*d2r} ${0*d2r}"/>
+    <origin xyz="0.76574 -0.570 0.577" rpy="${0*d2r} ${-110*d2r} ${-90*d2r}"/>
   </xacro:thruster_macro>
   <xacro:thruster_macro namespace="${namespace}" thruster_id="4">
