Commit message: add publisher to rexrov launch

File: uuv_descriptions/urdf/rexrov.gazebo.xacro (robot description, xacro)
@@ -20,5 +20,5 @@
     <xacro:property name="cob" value="0.0 0.0 0.3"/>
     <!-- Volume, see p.31 in Berg2012 -->
-    <xacro:property name="volume" value="1.83826"/>
+    <xacro:property name="volume" value="4.01461"/>
     <xacro:macro name="rexrov_hydro_model" params="namespace">
         <link name="${namespace}/base_link">
@@ -26,7 +26,7 @@
             <volume>${volume}</volume>
             <box>
-                <width>1.5</width>
-                <length>2.6</length>
-                <height>1.6</height>
+                <width>1.905</width>
+                <length>3.598</length>
+                <height>2.673</height>
             </box>
             <center_of_buoyancy>${cob}</center_of_buoyancy>

File: uuv_descriptions/urdf/rexrov_base.xacro (robot description, xacro)
@@ -30,5 +30,5 @@
   <xacro:property name="prop_mesh_file" value="file://$(find uuv_descriptions)/meshes/prop.dae"/>
   <!-- Mass, see p.28 in Berg2012 -->
-  <xacro:property name="mass" value="1862.87"/>
+  <xacro:property name="mass" value="4217.66"/>
   <xacro:macro name="rexrov_base" params="namespace *gazebo inertial_reference_frame">
     <!-- base_link according to ROS conventions: x forward, z up -->

Commit message: fix motors height

File: uuv_descriptions/urdf/rexrov.gazebo.xacro (robot description, xacro)
@@ -28,5 +28,5 @@
                 <width>1.905</width>
                 <length>3.598</length>
-                <height>2.673</height>
+                <height>2.049</height>
             </box>
             <center_of_buoyancy>${cob}</center_of_buoyancy>

File: uuv_descriptions/urdf/rexrov_actuators.xacro (robot description, xacro)
@@ -27,26 +27,26 @@
   </xacro:macro>
   <xacro:thruster_macro namespace="${namespace}" thruster_id="0">
-    <origin xyz="-0.76574 0.570 0.1577" rpy="${0*d2r} ${70*d2r} ${0*d2r}"/>
+    <origin xyz="-0.76574 0.570 0.577" rpy="${0*d2r} ${70*d2r} ${0*d2r}"/>
   </xacro:thruster_macro>
   <xacro:thruster_macro namespace="${namespace}" thruster_id="1">
-    <origin xyz="-0.76574 -0.570 0.1577" rpy="${0*d2r} ${-70*d2r} ${0*d2r}"/>
+    <origin xyz="-0.76574 -0.570 0.577" rpy="${0*d2r} ${-70*d2r} ${0*d2r}"/>
   </xacro:thruster_macro>
   <xacro:thruster_macro namespace="${namespace}" thruster_id="2">
-    <origin xyz="0.76574 0.570 0.1577" rpy="${0*d2r} ${110*d2r} ${0*d2r}"/>
+    <origin xyz="0.76574 0.570 0.577" rpy="${0*d2r} ${110*d2r} ${0*d2r}"/>
   </xacro:thruster_macro>
   <xacro:thruster_macro namespace="${namespace}" thruster_id="3">
-    <origin xyz="0.76574 -0.570 0.1577" rpy="${0*d2r} ${-110*d2r} ${0*d2r}"/>
+    <origin xyz="0.76574 -0.570 0.577" rpy="${0*d2r} ${-110*d2r} ${0*d2r}"/>
   </xacro:thruster_macro>
   <xacro:thruster_macro namespace="${namespace}" thruster_id="4">
-    <origin xyz="-1.19239 0.56425 0.94606" rpy="${0*d2r} ${0*d2r} ${45*d2r}"/>
+    <origin xyz="-1.19239 0.56425 -0.054" rpy="${0*d2r} ${0*d2r} ${45*d2r}"/>
   </xacro:thruster_macro>
   <xacro:thruster_macro namespace="${namespace}" thruster_id="5">
-    <origin xyz="-1.19239 -0.56425 0.94606" rpy="${0*d2r} ${0*d2r} ${-45*d2r}"/>
+    <origin xyz="-1.19239 -0.56425 -0.054" rpy="${0*d2r} ${0*d2r} ${-45*d2r}"/>
   </xacro:thruster_macro>
   <xacro:thruster_macro namespace="${namespace}" thruster_id="6">
-    <origin xyz="1.22921 0.56425 0.94606" rpy="${0*d2r} ${0*d2r} ${135*d2r}"/>
+    <origin xyz="1.22921 0.56425 -0.054" rpy="${0*d2r} ${0*d2r} ${135*d2r}"/>
   </xacro:thruster_macro>
   <xacro:thruster_macro namespace="${namespace}" thruster_id="7">
-    <origin xyz="1.229215 -0.56425 0.94606" rpy="${0*d2r} ${0*d2r} ${-135*d2r}"/>
+    <origin xyz="1.229215 -0.56425 -0.054" rpy="${0*d2r} ${0*d2r} ${-135*d2r}"/>
   </xacro:thruster_macro>
 </robot>

File: uuv_descriptions/urdf/rexrov_base.xacro (robot description, xacro)
@@ -39,10 +39,4 @@
         <inertia ixx="2760.99" ixy="29.02" ixz="20.94" iyy="5161.46" iyz="29.39" izz="4332.90"/>
       </inertial>
-      <visual>
-        <origin xyz="0 0 0" rpy="0 0 0"/>
-        <geometry>
-          <mesh filename="${visual_mesh_file}" scale="1.4 1.27 1.67"/>
-        </geometry>
-      </visual>
       <!-- bottom plate -->
       <collision>
@@ -60,9 +54,9 @@
       <collision>
         <origin xyz="-0.20 0.90 -0.15" rpy="0 0 0"/>
-        <geometry><box size="3.40 0.10 1.50"/></geometry>
+        <geometry><box size="3.40 0.10 1.9"/></geometry>
       </collision>
       <collision>
         <origin xyz="-0.20 -0.90 -0.15" rpy="0 0 0"/>
-        <geometry><box size="3.40 0.10 1.50"/></geometry>
+        <geometry><box size="3.40 0.10 1.9"/></geometry>
       </collision>
     </link>

Commit message: RMK model and state publisher (#1)
* create topics

* template for publishwer

* add speed position and acceleration topics

* add publisher to packages

* add publisher to packages

* add publisher to rexrov launch

* change inertia

* change thrusters positions

* fix motors height

* change proportions

* fix thruster angles

* change rotor constant

* update readme

* set joystick teleop for thrustmaster

* add bottom sonar

* publish depth

* add upper sonar

* altitude publisher

File: uuv_descriptions/urdf/rexrov.gazebo.xacro (robot description, xacro)
@@ -20,5 +20,5 @@
     <xacro:property name="cob" value="0.0 0.0 0.3"/>
     <!-- Volume, see p.31 in Berg2012 -->
-    <xacro:property name="volume" value="1.83826"/>
+    <xacro:property name="volume" value="4.01461"/>
     <xacro:macro name="rexrov_hydro_model" params="namespace">
         <link name="${namespace}/base_link">
@@ -26,7 +26,7 @@
             <volume>${volume}</volume>
             <box>
-                <width>1.5</width>
-                <length>2.6</length>
-                <height>1.6</height>
+                <width>1.905</width>
+                <length>3.598</length>
+                <height>2.049</height>
             </box>
             <center_of_buoyancy>${cob}</center_of_buoyancy>

File: uuv_descriptions/urdf/rexrov_actuators.xacro (robot description, xacro)
@@ -21,32 +21,32 @@
       thruster_id="${thruster_id}"
       mesh_filename="${prop_mesh_file}"
-      dyn_time_constant="0.05"
-      rotor_constant="0.00031">
+      dyn_time_constant="0.2"
+      rotor_constant="0.00124">
       <xacro:insert_block name="origin"/>
     </xacro:thruster_module_first_order_basic_fcn_macro>
   </xacro:macro>
-  <xacro:thruster_macro namespace="${namespace}" thruster_id="0">
-    <origin xyz="-0.890895 0.334385 0.528822" rpy="${0*d2r} ${-74.53*d2r} ${-53.21*d2r}"/>
+ <xacro:thruster_macro namespace="${namespace}" thruster_id="0">
+    <origin xyz="-0.76574 0.570 0.577" rpy="${0*d2r} ${-70*d2r} ${-90*d2r}"/>
   </xacro:thruster_macro>
   <xacro:thruster_macro namespace="${namespace}" thruster_id="1">
-    <origin xyz="-0.890895 -0.334385 0.528822" rpy="${0*d2r} ${-74.53*d2r} ${53.21*d2r}"/>
+    <origin xyz="-0.76574 -0.570 0.577" rpy="${0*d2r} ${-70*d2r} ${90*d2r}"/>
   </xacro:thruster_macro>
   <xacro:thruster_macro namespace="${namespace}" thruster_id="2">
-    <origin xyz="0.890895 0.334385 0.528822" rpy="${0*d2r} ${-105.47*d2r} ${53.21*d2r}"/>
+    <origin xyz="0.76574 0.570 0.577" rpy="${0*d2r} ${-110*d2r} ${90*d2r}"/>
   </xacro:thruster_macro>
   <xacro:thruster_macro namespace="${namespace}" thruster_id="3">
-    <origin xyz="0.890895 -0.334385 0.528822" rpy="${0*d2r} ${-105.47*d2r} ${-53.21*d2r}"/>
+    <origin xyz="0.76574 -0.570 0.577" rpy="${0*d2r} ${-110*d2r} ${-90*d2r}"/>
   </xacro:thruster_macro>
   <xacro:thruster_macro namespace="${namespace}" thruster_id="4">
-    <origin xyz="-0.412125 0.505415 0.129" rpy="${0*d2r} ${0*d2r} ${45*d2r}"/>
+    <origin xyz="-1.19239 0.56425 -0.054" rpy="${0*d2r} ${0*d2r} ${45*d2r}"/>
   </xacro:thruster_macro>
   <xacro:thruster_macro namespace="${namespace}" thruster_id="5">
-    <origin xyz="-0.412125 -0.505415 0.129" rpy="${0*d2r} ${0*d2r} ${-45*d2r}"/>
+    <origin xyz="-1.19239 -0.56425 -0.054" rpy="${0*d2r} ${0*d2r} ${-45*d2r}"/>
   </xacro:thruster_macro>
   <xacro:thruster_macro namespace="${namespace}" thruster_id="6">
-    <origin xyz="0.412125 0.505415 0.129" rpy="${0*d2r} ${0*d2r} ${135*d2r}"/>
+    <origin xyz="1.22921 0.56425 -0.054" rpy="${0*d2r} ${0*d2r} ${135*d2r}"/>
   </xacro:thruster_macro>
   <xacro:thruster_macro namespace="${namespace}" thruster_id="7">
-    <origin xyz="0.412125 -0.505415 0.129" rpy="${0*d2r} ${0*d2r} ${-135*d2r}"/>
+    <origin xyz="1.229215 -0.56425 -0.054" rpy="${0*d2r} ${0*d2r} ${-135*d2r}"/>
   </xacro:thruster_macro>
 </robot>

File: uuv_descriptions/urdf/rexrov_base.xacro (robot description, xacro)
@@ -30,5 +30,5 @@
   <xacro:property name="prop_mesh_file" value="file://$(find uuv_descriptions)/meshes/prop.dae"/>
   <!-- Mass, see p.28 in Berg2012 -->
-  <xacro:property name="mass" value="1862.87"/>
+  <xacro:property name="mass" value="4217.66"/>
   <xacro:macro name="rexrov_base" params="namespace *gazebo inertial_reference_frame">
     <!-- base_link according to ROS conventions: x forward, z up -->
@@ -37,32 +37,32 @@
         <mass value="${mass}"/>
         <origin xyz="0 0 0"/>
-        <inertia ixx="525.39" ixy="1.44" ixz="33.41" iyy="794.20" iyz="2.6" izz="691.23"/>
+        <inertia ixx="2760.99" ixy="29.02" ixz="20.94" iyy="5161.46" iyz="29.39" izz="4332.90"/>
       </inertial>
       <visual>
         <origin xyz="0 0 0" rpy="0 0 0"/>
         <geometry>
-          <mesh filename="${visual_mesh_file}" scale="1 1 1"/>
+          <mesh filename="${visual_mesh_file}" scale="1.4 1.27 1.25"/>
         </geometry>
       </visual>
       <!-- bottom plate -->
       <collision>
-        <origin xyz="0 0 -0.75" rpy="0 0 0"/>
+        <origin xyz="0 0 -0.85" rpy="0 0 0"/>
         <geometry>
-          <box size="2.56 1.50 0.10"/>
+          <box size="3.598 1.905 0.10"/>
         </geometry>
       </collision>
       <!-- top plate -->
       <collision>
-        <origin xyz="0 0 0.60" rpy="0 0 0"/>
-        <geometry><box size="2.56 1.50 0.40"/></geometry>
+        <origin xyz="0 0 0.70" rpy="0 0 0"/>
+        <geometry><box size="3.598 1.905 0.40"/></geometry>
       </collision>
       <!-- left / right sides -->
       <collision>
-        <origin xyz="-0.20 0.70 -0.15" rpy="0 0 0"/>
-        <geometry><box size="2.20 0.10 1.10"/></geometry>
+        <origin xyz="-0.20 0.90 -0.15" rpy="0 0 0"/>
+        <geometry><box size="3.40 0.10 1.9"/></geometry>
       </collision>
       <collision>
-        <origin xyz="-0.20 -0.70 -0.15" rpy="0 0 0"/>
-        <geometry><box size="2.20 0.10 1.10"/></geometry>
+        <origin xyz="-0.20 -0.90 -0.15" rpy="0 0 0"/>
+        <geometry><box size="3.40 0.10 1.9"/></geometry>
       </collision>
     </link>

File: uuv_descriptions/urdf/rexrov_sensors.xacro (robot description, xacro)
@@ -20,4 +20,12 @@
     <origin xyz="-1.4 0 -0.312" rpy="0 ${0.5*pi} 0"/>
   </xacro:default_dvl_macro>
+<!-- Down Sonar -->
+  <xacro:sidescan_sonar namespace="${namespace}" parent_link="${namespace}/base_link" suffix="down">
+  <origin xyz="0 0 -0.92" rpy="0 ${0.5*pi} 0"/>
+  </xacro:sidescan_sonar>
+<!-- Up Sonar -->
+  <xacro:sidescan_sonar namespace="${namespace}" parent_link="${namespace}/base_link" suffix="up">
+  <origin xyz="0 0 0.92" rpy="0 ${-0.5*pi} 0"/>
+  </xacro:sidescan_sonar>
   <!-- Magnetometer  -->
   <xacro:default_magnetometer namespace="${namespace}" parent_link="${namespace}/base_link"/>
